File: pcb/lmx2594/lmx2594.sch (KiCad schematic (older format))
At the start: 80 parts, among them J1 Conn_Coaxial, J2 Conn_Coaxial, J3 Conn_01x13_Male, J4 Conn_Coaxial, J5 Conn_Coaxial, J6 Conn_Coaxial, J7 Conn_Coaxial, J8 Conn_Coaxial, J9 Conn_Coaxial, U1 L7812, U2 TPS62150, U3 lmx254

Commit message: More work on layout
Parts:
- C11, C12, C13, C14, C17, C18, C19, C2, C20, C21, C22, C23, C24, C25, C26, C27, C28, C29, C3, C30, C31, C32, C33, C34, C35, C36, C37, C38, C39, C40, C41, C42, C43, C6, C7, C8, L7, L8: footprint Capacitors_SMD:C_0603_HandSoldering -> Capacitors_SMD:C_0603
- R1, R10, R11, R12, R13, R14, R15, R16, R17, R18, R19, R2, R20, R21, R22, R4, R5, R6, R7, R9: footprint Resistors_SMD:R_0603_HandSoldering -> Resistors_SMD:R_0603
Connections:
- net SYSREFREQ_S is gone; now on net SDI: J3.10 (Pin_10)
- net 12V: no longer J3.2 (Pin_2), R5.2
- net CE: now also J3.6 (Pin_6); no longer J3.5 (Pin_5)
- net CSB: now also J3.12 (Pin_12); no longer J3.6 (Pin_6)
- net MUX: now also J3.11 (Pin_11); no longer J3.13 (Pin_13)
- net RAMPCLK: now also J3.8 (Pin_8); no longer J3.11 (Pin_11)
- net RAMPDIR: now also J3.7 (Pin_7); no longer J3.12 (Pin_12)
- net SCK: now also J3.9 (Pin_9); no longer J3.8 (Pin_8)
- net SDI: no longer J3.7 (Pin_7)
- net SYNC: now also R20.1, R22.1; no longer R18.1, R19.1
- net SYNC_S: now also J3.5 (Pin_5), R20.2; no longer J3.9 (Pin_9), R18.2
- net SYSREFREQ: now also R18.1, R19.1; no longer R20.1, R22.1
- net SYSREF_REQ_S: now also J3.13 (Pin_13), R18.2; no longer R20.2
- net VCC: no longer J3.4 (Pin_4)
- net SW: now reaches L4.1, U2.1 (SW), U2.2 (SW), U2.3 (SW)
- net 3V3: now reaches C12.1, L1.1, L4.2, L5.1, R2.2, R6.1, R7.2, U2.14 (VOS), U2.7 (FSW)
- net 3V3: now also J3.4 (Pin_4)
- net CPOUT: now reaches C30.1, C31.1, R15.1, U3.12 (CPOUT)
- net RFOUT_B_N: now reaches C26.2, R13.1, U3.18 (RFOUTBM)
- net RFOUT_B_P: now reaches C33.2, R16.2, U3.19 (RFOUTBP)
- net RFOUT_A_N: now reaches C20.2, R12.2, U3.22 (RFOUTAM)
- net RFOUT_A_P: now reaches C17.2, R11.1, U3.23 (RFOUTAP)
- net VTUNE: now reaches C28.1, R14.2, U3.35 (VTUNE)
- net OSCIN_P: now reaches C41.1, U3.8 (OSCINP)
- net OSCIN_N: now reaches C43.1, U3.9 (OSCINM)
- net RFA_BIAS: now reaches C18.2, L7.1, R11.2, R12.1
- net 12V_unfilt: now reaches C3.1, C4.1, L3.1, R1.2, U1.3 (OUT)
- net 12V_unfilt: now also J3.2 (Pin_2), R5.2
- net RFB_BIAS: now reaches C27.2, L8.1, R13.2, R16.1
Other:
- moved on the sheet: J6, J8, R18, R19, R20, R22

Commit message: Layout sort is probably done, can make something nicer with powerplanes but i do not think it is needed. Silkscreen must also be fixed
Parts:
- R1, R10, R11, R12, R13, R14, R15, R16, R17, R18, R19, R2, R20, R21, R22, R4, R5, R6, R7, R9: footprint Resistors_SMD:R_0603 -> Capacitors_SMD:C_0603
Changed lines of the file:
@@
 EESchema Schematic File Version 4
+LIBS:lmx2594-cache
 EELAYER 26 0
 EELAYER END
@@
 F 0 "R11" H 9820 2996 50  0000 L CNN
 F 1 "50" H 9820 2905 50  0000 L CNN
-F 2 "Resistors_SMD:R_0603" V 9680 2950 50  0001 C CNN
+F 2 "Capacitors_SMD:C_0603" V 9680 2950 50  0001 C CNN
 F 3 "~" H 9750 2950 50  0001 C CNN
 	1    9750 2950
@@
 F 0 "R12" H 9820 3396 50  0000 L CNN
 F 1 "50" H 9820 3305 50  0000 L CNN
-F 2 "Resistors_SMD:R_0603" V 9680 3350 50  0001 C CNN
+F 2 "Capacitors_SMD:C_0603" V 9680 3350 50  0001 C CNN
 F 3 "~" H 9750 3350 50  0001 C CNN
 	1    9750 3350
@@
 F 0 "R21" H 3170 6096 50  0000 L CNN
 F 1 "100" H 3170 6005 50  0000 L CNN
-F 2 "Resistors_SMD:R_0603" V 3030 6050 50  0001 C CNN
+F 2 "Capacitors_SMD:C_0603" V 3030 6050 50  0001 C CNN
 F 3 "~" H 3100 6050 50  0001 C CNN
 	1    3100 6050
@@
 F 0 "R6" H 5920 1696 50  0000 L CNN
 F 1 "562K" H 5920 1605 50  0000 L CNN
-F 2 "Resistors_SMD:R_0603" V 5780 1650 50  0001 C CNN
+F 2 "Capacitors_SMD:C_0603" V 5780 1650 50  0001 C CNN
 F 3 "~" H 5850 1650 50  0001 C CNN
 	1    5850 1650
@@
 F 0 "R10" H 5920 2096 50  0000 L CNN
 F 1 "180K" H 5920 2005 50  0000 L CNN
-F 2 "Resistors_SMD:R_0603" V 5780 2050 50  0001 C CNN
+F 2 "Capacitors_SMD:C_0603" V 5780 2050 50  0001 C CNN
 F 3 "~" H 5850 2050 50  0001 C CNN
 	1    5850 2050
@@
 F 0 "R2" V 6693 1000 50  0000 C CNN
 F 1 "0" V 6784 1000 50  0000 C CNN
-F 2 "Resistors_SMD:R_0603" V 6830 1000 50  0001 C CNN
+F 2 "Capacitors_SMD:C_0603" V 6830 1000 50  0001 C CNN
 F 3 "~" H 6900 1000 50  0001 C CNN
 	1    6900 1000
@@
 F 0 "R7" V 6693 1800 50  0000 C CNN
 F 1 "0" V 6784 1800 50  0000 C CNN
-F 2 "Resistors_SMD:R_0603" V 6830 1800 50  0001 C CNN
+F 2 "Capacitors_SMD:C_0603" V 6830 1800 50  0001 C CNN
 F 3 "~" H 6900 1800 50  0001 C CNN
 	1    6900 1800
@@
 F 0 "R13" H 9820 4396 50  0000 L CNN
 F 1 "50" H 9820 4305 50  0000 L CNN
-F 2 "Resistors_SMD:R_0603" V 9680 4350 50  0001 C CNN
+F 2 "Capacitors_SMD:C_0603" V 9680 4350 50  0001 C CNN
 F 3 "~" H 9750 4350 50  0001 C CNN
 	1    9750 4350
@@
 F 0 "R16" H 9820 4796 50  0000 L CNN
 F 1 "50" H 9820 4705 50  0000 L CNN
-F 2 "Resistors_SMD:R_0603" V 9680 4750 50  0001 C CNN
+F 2 "Capacitors_SMD:C_0603" V 9680 4750 50  0001 C CNN
 F 3 "~" H 9750 4750 50  0001 C CNN
 	1    9750 4750
@@
 F 0 "R14" V 7543 4500 50  0000 C CNN
 F 1 "18" V 7634 4500 50  0000 C CNN
-F 2 "Resistors_SMD:R_0603" V 7680 4500 50  0001 C CNN
+F 2 "Capacitors_SMD:C_0603" V 7680 4500 50  0001 C CNN
 F 3 "~" H 7750 4500 50  0001 C CNN
 	1    7750 4500
@@
 F 0 "R15" V 7943 4500 50  0000 C CNN
 F 1 "0" V 8034 4500 50  0000 C CNN
-F 2 "Resistors_SMD:R_0603" V 8080 4500 50  0001 C CNN
+F 2 "Capacitors_SMD:C_0603" V 8080 4500 50  0001 C CNN
 F 3 "~" H 8150 4500 50  0001 C CNN
 	1    8150 4500
@@
 F 0 "R17" H 8330 5004 50  0000 R CNN
 F 1 "68" H 8330 5095 50  0000 R CNN
-F 2 "Resistors_SMD:R_0603" V 8330 5050 50  0001 C CNN
+F 2 "Capacitors_SMD:C_0603" V 8330 5050 50  0001 C CNN
 F 3 "~" H 8400 5050 50  0001 C CNN
 	1    8400 5050
@@
 F 0 "R4" V 9493 1200 50  0000 C CNN
 F 1 "150" V 9584 1200 50  0000 C CNN
-F 2 "Resistors_SMD:R_0603" V 9630 1200 50  0001 C CNN
+F 2 "Capacitors_SMD:C_0603" V 9630 1200 50  0001 C CNN
 F 3 "~" H 9700 1200 50  0001 C CNN
 	1    9700 1200
@@
 F 0 "R5" V 9493 1500 50  0000 C CNN
 F 1 "1k" V 9584 1500 50  0000 C CNN
-F 2 "Resistors_SMD:R_0603" V 9630 1500 50  0001 C CNN
+F 2 "Capacitors_SMD:C_0603" V 9630 1500 50  0001 C CNN
 F 3 "~" H 9700 1500 50  0001 C CNN
 	1    9700 1500
@@
 F 0 "R9" V 9493 1800 50  0000 C CNN
 F 1 "150" V 9584 1800 50  0000 C CNN
-F 2 "Resistors_SMD:R_0603" V 9630 1800 50  0001 C CNN
+F 2 "Capacitors_SMD:C_0603" V 9630 1800 50  0001 C CNN
 F 3 "~" H 9700 1800 50  0001 C CNN
 	1    9700 1800
@@
 F 0 "R22" V 9193 5550 50  0000 C CNN
 F 1 "0" V 9284 5550 50  0000 C CNN
-F 2 "Resistors_SMD:R_0603" V 9330 5550 50  0001 C CNN
+F 2 "Capacitors_SMD:C_0603" V 9330 5550 50  0001 C CNN
 F 3 "~" H 9400 5550 50  0001 C CNN
 	1    9400 5550
@@
 F 0 "R19" V 9193 6150 50  0000 C CNN
 F 1 "0" V 9284 6150 50  0000 C CNN
-F 2 "Resistors_SMD:R_0603" V 9330 6150 50  0001 C CNN
+F 2 "Capacitors_SMD:C_0603" V 9330 6150 50  0001 C CNN
 F 3 "~" H 9400 6150 50  0001 C CNN
 	1    9400 6150
@@
 F 0 "R18" V 9193 5850 50  0000 C CNN
 F 1 "0" V 9284 5850 50  0000 C CNN
-F 2 "Resistors_SMD:R_0603" V 9330 5850 50  0001 C CNN
+F 2 "Capacitors_SMD:C_0603" V 9330 5850 50  0001 C CNN
 F 3 "~" H 9400 5850 50  0001 C CNN
 	1    9400 5850
@@
 F 0 "R20" V 9193 5250 50  0000 C CNN
 F 1 "0" V 9284 5250 50  0000 C CNN
-F 2 "Resistors_SMD:R_0603" V 9330 5250 50  0001 C CNN
+F 2 "Capacitors_SMD:C_0603" V 9330 5250 50  0001 C CNN
 F 3 "~" H 9400 5250 50  0001 C CNN
 	1    9400 5250
@@
 F 0 "R1" V 2943 650 50  0000 C CNN
 F 1 "0" V 3034 650 50  0000 C CNN
-F 2 "Resistors_SMD:R_0603" V 3080 650 50  0001 C CNN
+F 2 "Capacitors_SMD:C_0603" V 3080 650 50  0001 C CNN
 F 3 "~" H 3150 650 50  0001 C CNN
 	1    3150 650

Commit message: Added single ended terminations to osci
Parts:
- added R? (x2): 50, Capacitors_SMD:C_0603, symbol Device:R
Connections:
- net GND: now also R?.1, R?.2
- net at C40.1, C41.2, R21.1: now also R?.2
- net at C42.1, C43.2, R21.2: now also R?.1
Changed lines of the file:
@@
 Connection ~ 3100 6350
 Wire Wire Line
-	3100 6350 3250 6350
+	3100 6350 3150 6350
 Wire Wire Line
 	3100 5900 3100 5750
 Connection ~ 3100 5750
 Wire Wire Line
-	3100 5750 3250 5750
+	3100 5750 3150 5750
 Wire Wire Line
 	3550 5750 4950 5750
@@
 Text Label 9200 1500 0    50   ~ 0
 12V_unfilt
+$Comp
+L Device:R R?
+U 1 1 5CD0456C
+P 3150 6500
+F 0 "R?" H 3220 6546 50  0000 L CNN
+F 1 "50" H 3220 6455 50  0000 L CNN
+F 2 "Capacitors_SMD:C_0603" V 3080 6500 50  0001 C CNN
+F 3 "~" H 3150 6500 50  0001 C CNN
+	1    3150 6500
+	1    0    0    -1
+$EndComp
+Connection ~ 3150 6350
+Wire Wire Line
+	3150 6350 3250 6350
+$Comp
+L Device:R R?
+U 1 1 5CD047D2
+P 3150 5600
+F 0 "R?" H 3220 5646 50  0000 L CNN
+F 1 "50" H 3220 5555 50  0000 L CNN
+F 2 "Capacitors_SMD:C_0603" V 3080 5600 50  0001 C CNN
+F 3 "~" H 3150 5600 50  0001 C CNN
+	1    3150 5600
+	1    0    0    -1
+$EndComp
+Connection ~ 3150 5750
+Wire Wire Line
+	3150 5750 3250 5750
+$Comp
+L power:GND #PWR?
+U 1 1 5CD04904
+P 3150 6700
+F 0 "#PWR?" H 3150 6450 50  0001 C CNN
+F 1 "GND" H 3155 6527 50  0000 C CNN
+F 2 "" H 3150 6700 50  0001 C CNN
+F 3 "" H 3150 6700 50  0001 C CNN
+	1    3150 6700
+	1    0    0    -1
+$EndComp
+$Comp
+L power:GND #PWR?
+U 1 1 5CD049B3
+P 3050 5450
+F 0 "#PWR?" H 3050 5200 50  0001 C CNN
+F 1 "GND" H 3055 5277 50  0000 C CNN
+F 2 "" H 3050 5450 50  0001 C CNN
+F 3 "" H 3050 5450 50  0001 C CNN
+	1    3050 5450
+	1    0    0    -1
+$EndComp
+Wire Wire Line
+	3150 5450 3050 5450
+Wire Wire Line
+	3150 6650 3150 6700
 $EndSCHEMATC

Commit message: Tidying up a bit and added pullup on CE
Parts:
- added R?: 10K, Capacitors_SMD:C_0603, symbol Device:R
- gave numbers to parts that had none: 2
Connections:
- net CE: now also R?.2
- net VCC: now also R?.1
Changed lines of the file:
@@
 	6450 6150 6500 6150
-Wire Wire Line
-	5400 4300 5250 4300
 Wire Wire Line
 	5400 4400 5250 4400
@@
 12V_unfilt
 $Comp
-L Device:R R?
+L Device:R R8
 U 1 1 5CD0456C
 P 3150 6500
-F 0 "R?" H 3220 6546 50  0000 L CNN
+F 0 "R8" H 3220 6546 50  0000 L CNN
 F 1 "50" H 3220 6455 50  0000 L CNN
 F 2 "Capacitors_SMD:C_0603" V 3080 6500 50  0001 C CNN
@@
 	3150 6350 3250 6350
 $Comp
-L Device:R R?
+L Device:R R3
 U 1 1 5CD047D2
 P 3150 5600
-F 0 "R?" H 3220 5646 50  0000 L CNN
+F 0 "R3" H 3220 5646 50  0000 L CNN
 F 1 "50" H 3220 5555 50  0000 L CNN
 F 2 "Capacitors_SMD:C_0603" V 3080 5600 50  0001 C CNN
@@
 	3150 5750 3250 5750
 $Comp
-L power:GND #PWR?
+L power:GND #PWR0109
 U 1 1 5CD04904
 P 3150 6700
-F 0 "#PWR?" H 3150 6450 50  0001 C CNN
+F 0 "#PWR0109" H 3150 6450 50  0001 C CNN
 F 1 "GND" H 3155 6527 50  0000 C CNN
 F 2 "" H 3150 6700 50  0001 C CNN
@@
 $EndComp
 $Comp
-L power:GND #PWR?
+L power:GND #PWR0110
 U 1 1 5CD049B3
 P 3050 5450
-F 0 "#PWR?" H 3050 5200 50  0001 C CNN
+F 0 "#PWR0110" H 3050 5200 50  0001 C CNN
 F 1 "GND" H 3055 5277 50  0000 C CNN
 F 2 "" H 3050 5450 50  0001 C CNN
@@
 Wire Wire Line
 	3150 6650 3150 6700
+$Comp
+L Device:R R?
+U 1 1 5CD25BC9
+P 5000 4300
+F 0 "R?" V 4793 4300 50  0000 C CNN
+F 1 "10K" V 4884 4300 50  0000 C CNN
+F 2 "Capacitors_SMD:C_0603" V 4930 4300 50  0001 C CNN
+F 3 "~" H 5000 4300 50  0001 C CNN
+	1    5000 4300
+	0    -1   1    0
+$EndComp
+Wire Wire Line
+	5150 4300 5400 4300
+Wire Wire Line
+	4850 4300 4650 4300
+Text Label 4650 4300 0    50   ~ 0
+VCC
 $EndSCHEMATC

Commit message: More review of schematic
Parts:
- gave numbers to parts that had none: 1
Changed lines of the file:
@@
 	3150 6650 3150 6700
 $Comp
-L Device:R R?
+L Device:R R23
 U 1 1 5CD25BC9
 P 5000 4300
-F 0 "R?" V 4793 4300 50  0000 C CNN
+F 0 "R23" V 4793 4300 50  0000 C CNN
 F 1 "10K" V 4884 4300 50  0000 C CNN
 F 2 "Capacitors_SMD:C_0603" V 4930 4300 50  0001 C CNN

Commit message: Review, fixed vbuf and added pg led
Parts:
- added D4: LED, LEDs:LED_0805_HandSoldering, symbol Device:LED
- added R24: 150, Capacitors_SMD:C_0603, symbol Device:R
- added R25, R26: 0, Capacitors_SMD:C_0603, symbol Device:R
Connections:
- net 3V3: now also R9.2, R24.2
- net VCC: now also R26.1; no longer C19.2, R9.2, U3.21 (VCCBUF)
- net VRF: now also R25.1
- net PG: now reaches U2.4 (PG)
- net PG: now also D4.1 (K)
- new net: C19.2, R25.2, R26.2, U3.21 (VCCBUF)
- new net: D4.2 (A), R24.1
Other:
- note added: "Add LED for PG on regulator"
- note added: "Use VRF instead"
Changed lines of the file:
@@
 	5400 3300 5050 3300
 Connection ~ 5400 3300
-Text Label 5050 3300 0    50   ~ 0
+Text Label 4550 3300 0    50   ~ 0
 VCC
 Wire Wire Line
 	5350 4100 5350 4000
-Wire Wire Line
-	5350 3600 5400 3600
 Connection ~ 5350 4100
 Wire Wire Line
 	5350 4100 5000 4100
-Connection ~ 5400 3600
 Connection ~ 5350 4000
 Wire Wire Line
@@
 Wire Wire Line
 	5350 3700 5300 3700
-Wire Wire Line
-	5350 3700 5350 3600
 Wire Wire Line
 	10400 2800 10150 2800
@@
 Text Label 9200 1200 0    50   ~ 0
 MUX
-Text Label 9200 1800 0    50   ~ 0
-VCC
 Text Label 1550 3750 0    50   ~ 0
 CE
@@
 Text Label 4650 4300 0    50   ~ 0
 VCC
+Text Notes 9250 2400 0    50   ~ 0
+Add LED for PG on regulator
+Text Notes 5750 3200 0    50   ~ 0
+Use VRF instead
+$Comp
+L Device:R R25
+U 1 1 5CFBE008
+P 4900 3000
+F 0 "R25" V 4693 3000 50  0000 C CNN
+F 1 "0" V 4784 3000 50  0000 C CNN
+F 2 "Capacitors_SMD:C_0603" V 4830 3000 50  0001 C CNN
+F 3 "~" H 4900 3000 50  0001 C CNN
+	1    4900 3000
+	0    -1   1    0
+$EndComp
+$Comp
+L Device:R R26
+U 1 1 5CFBE134
+P 4900 3300
+F 0 "R26" V 4693 3300 50  0000 C CNN
+F 1 "0" V 4784 3300 50  0000 C CNN
+F 2 "Capacitors_SMD:C_0603" V 4830 3300 50  0001 C CNN
+F 3 "~" H 4900 3300 50  0001 C CNN
+	1    4900 3300
+	0    -1   1    0
+$EndComp
+Wire Wire Line
+	5050 3300 5050 3000
+Connection ~ 5050 3300
+Wire Wire Line
+	4750 3000 4550 3000
+Wire Wire Line
+	4750 3300 4550 3300
+Text Label 4550 3000 0    50   ~ 0
+VRF
+$Comp
+L Device:R R24
+U 1 1 5CFEBE2A
+P 9700 2100
+F 0 "R24" V 9493 2100 50  0000 C CNN
+F 1 "150" V 9584 2100 50  0000 C CNN
+F 2 "Capacitors_SMD:C_0603" V 9630 2100 50  0001 C CNN
+F 3 "~" H 9700 2100 50  0001 C CNN
+	1    9700 2100
+	0    1    1    0
+$EndComp
+$Comp
+L Device:LED D4
+U 1 1 5CFEBE30
+P 10100 2100
+F 0 "D4" H 10092 1845 50  0000 C CNN
+F 1 "LED" H 10092 1936 50  0000 C CNN
+F 2 "LEDs:LED_0805_HandSoldering" H 10100 2100 50  0001 C CNN
+F 3 "~" H 10100 2100 50  0001 C CNN
+	1    10100 2100
+	-1   0    0    1
+$EndComp
+Wire Wire Line
+	10350 2100 10250 2100
+Wire Wire Line
+	9950 2100 9850 2100
+Wire Wire Line
+	9550 2100 9200 2100
+Wire Wire Line
+	4850 1600 5200 1600
+Text Label 4950 1600 0    50   ~ 0
+PG
+Text Label 10350 2100 0    50   ~ 0
+PG
+Wire Wire Line
+	5350 3700 5350 3600
+Wire Wire Line
+	5350 3600 5000 3600
+Text Label 5000 3600 0    50   ~ 0
+VCC
+Text Label 9250 1800 0    50   ~ 0
+3V3
+Text Label 9250 2100 0    50   ~ 0
+3V3
 $EndSCHEMATC
